Commit message: changed package names in h1 urdf

File: dynamic_payload_analysis_core/examples/urdf/h1_description/urdf/h1.urdf (robot description, URDF)
Before this commit: robot h1_description, 25 links, 24 joints
Links:
- link left_ankle_link: geometry collision box size=0.28 0.03 0.024; visual mesh filename=package://dynamic_payload_analysis_core/examples/urdf/h1_de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
- link left_elbow_link: geometry collision cylinder length=0.09 radius=0.03; visual mesh filename=package://dynamic_payload_analysis_core/examples/urdf/h1_de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
- link left_hip_pitch_link: geometry collision cylinder length=0.2 radius=0.05; visual mesh filename=package://dynamic_payload_analysis_core/examples/urdf/h1_de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
- link left_hip_roll_link: geometry collision cylinder length=0.01 radius=0.02; visual mesh filename=package://dynamic_payload_analysis_core/examples/urdf/h1_de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
- link left_hip_yaw_link: geometry collision cylinder length=0.02 radius=0.01; visual mesh filename=package://dynamic_payload_analysis_core/examples/urdf/h1_de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
- link left_knee_link: geometry collision cylinder length=0.2 radius=0.05; visual mesh filename=package://dynamic_payload_analysis_core/examples/urdf/h1_de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
- link left_shoulder_pitch_link: geometry collision cylinder length=0.04 radius=0.03; visual mesh filename=package://dynamic_payload_analysis_core/examples/urdf/h1_de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
- link left_shoulder_roll_link: geometry collision cylinder length=0.01 radius=0.04; visual mesh filename=package://dynamic_payload_analysis_core/examples/urdf/h1_de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
- link left_shoulder_yaw_link: geometry collision cylinder length=0.01 radius=0.04; visual mesh filename=package://dynamic_payload_analysis_core/examples/urdf/h1_de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
- link logo_link: geometry visual mesh filename=package://dynamic_payload_analysis_core/examples/urdf/h1_de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
- link pelvis: geometry collision sphere radius=0.05; visual mesh filename=package://dynamic_payload_analysis_core/examples/urdf/h1_de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
- link right_ankle_link: geometry collision box size=0.28 0.03 0.024; visual mesh filename=package://dynamic_payload_analysis_core/examples/urdf/h1_de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
- link right_elbow_link: geometry collision cylinder length=0.09 radius=0.03; visual mesh filename=package://dynamic_payload_analysis_core/examples/urdf/h1_de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
- link right_hip_pitch_link: geometry collision cylinder length=0.2 radius=0.05; visual mesh filename=package://dynamic_payload_analysis_core/examples/urdf/h1_de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
- link right_hip_roll_link: geometry collision cylinder length=0.01 radius=0.02; visual mesh filename=package://dynamic_payload_analysis_core/examples/urdf/h1_de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
- link right_hip_yaw_link: geometry collision cylinder length=0.02 radius=0.01; visual mesh filename=package://dynamic_payload_analysis_core/examples/urdf/h1_de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
- link right_knee_link: geometry collision cylinder length=0.2 radius=0.05; visual mesh filename=package://dynamic_payload_analysis_core/examples/urdf/h1_de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
- link right_shoulder_pitch_link: geometry collision cylinder length=0.04 radius=0.03; visual mesh filename=package://dynamic_payload_analysis_core/examples/urdf/h1_de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
- link right_shoulder_roll_link: geometry collision cylinder length=0.01 radius=0.04; visual mesh filename=package://dynamic_payload_analysis_core/examples/urdf/h1_de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
- link right_shoulder_yaw_link: geometry collision cylinder length=0.01 radius=0.04; visual mesh filename=package://dynamic_payload_analysis_core/examples/urdf/h1_de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
- link torso_link: geometry collision box size=0.08 0.16 0.1; visual mesh filename=package://dynamic_payload_analysis_core/examples/urdf/h1_de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

File: dynamic_payload_analysis_core/examples/urdf/h1_description/urdf/h1_with_hand.urdf (robot description, URDF)
Before this commit: robot h1, 52 links, 51 joints
Links:
- link L_hand_base_link: geometry collision mesh filename=package://dynamic_payload_analysis_core/examples/urdf/h1_de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; visual mesh filename=package://dynamic_payload_analysis_core/examples/urdf/h1_de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
- link L_index_intermediate: geometry collision mesh filename=package://dynamic_payload_analysis_core/examples/urdf/h1_de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; visual mesh filename=package://dynamic_payload_analysis_core/examples/urdf/h1_de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
- link L_index_proximal: geometry collision mesh filename=package://dynamic_payload_analysis_core/examples/urdf/h1_de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; visual mesh filename=package://dynamic_payload_analysis_core/examples/urdf/h1_de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
- link L_middle_intermediate: geometry collision mesh filename=package://dynamic_payload_analysis_core/examples/urdf/h1_de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; visual mesh filename=package://dynamic_payload_analysis_core/examples/urdf/h1_de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
- link L_middle_proximal: geometry collision mesh filename=package://dynamic_payload_analysis_core/examples/urdf/h1_de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; visual mesh filename=package://dynamic_payload_analysis_core/examples/urdf/h1_de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
- link L_pinky_intermediate: geometry collision mesh filename=package://dynamic_payload_analysis_core/examples/urdf/h1_de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; visual mesh filename=package://dynamic_payload_analysis_core/examples/urdf/h1_de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
- link L_pinky_proximal: geometry collision mesh filename=package://dynamic_payload_analysis_core/examples/urdf/h1_de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; visual mesh filename=package://dynamic_payload_analysis_core/examples/urdf/h1_de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
- link L_ring_intermediate: geometry collision mesh filename=package://dynamic_payload_analysis_core/examples/urdf/h1_de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; visual mesh filename=package://dynamic_payload_analysis_core/examples/urdf/h1_de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
- link L_ring_proximal: geometry collision mesh filename=package://dynamic_payload_analysis_core/examples/urdf/h1_de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; visual mesh filename=package://dynamic_payload_analysis_core/examples/urdf/h1_de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
- link L_thumb_distal: geometry collision mesh filename=package://dynamic_payload_analysis_core/examples/urdf/h1_de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; visual mesh filename=package://dynamic_payload_analysis_core/examples/urdf/h1_de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
- link L_thumb_intermediate: geometry collision mesh filename=package://dynamic_payload_analysis_core/examples/urdf/h1_de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; visual mesh filename=package://dynamic_payload_analysis_core/examples/urdf/h1_de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
- link L_thumb_proximal: geometry collision mesh filename=package://dynamic_payload_analysis_core/examples/urdf/h1_de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; visual mesh filename=package://dynamic_payload_analysis_core/examples/urdf/h1_de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
- link L_thumb_proximal_base: geometry collision mesh filename=package://dynamic_payload_analysis_core/examples/urdf/h1_de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; visual mesh filename=package://dynamic_payload_analysis_core/examples/urdf/h1_de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
- link R_hand_base_link: geometry collision mesh filename=package://dynamic_payload_analysis_core/examples/urdf/h1_de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; visual mesh filename=package://dynamic_payload_analysis_core/examples/urdf/h1_de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
- link R_index_intermediate: geometry collision mesh filename=package://dynamic_payload_analysis_core/examples/urdf/h1_de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; visual mesh filename=package://dynamic_payload_analysis_core/examples/urdf/h1_de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
- link R_index_proximal: geometry collision mesh filename=package://dynamic_payload_analysis_core/examples/urdf/h1_de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; visual mesh filename=package://dynamic_payload_analysis_core/examples/urdf/h1_de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
- link R_middle_intermediate: geometry collision mesh filename=package://dynamic_payload_analysis_core/examples/urdf/h1_de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; visual mesh filename=package://dynamic_payload_analysis_core/examples/urdf/h1_de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
- link R_middle_proximal: geometry collision mesh filename=package://dynamic_payload_analysis_core/examples/urdf/h1_de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; visual mesh filename=package://dynamic_payload_analysis_core/examples/urdf/h1_de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
- link R_pinky_intermediate: geometry collision mesh filename=package://dynamic_payload_analysis_core/examples/urdf/h1_de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; visual mesh filename=package://dynamic_payload_analysis_core/examples/urdf/h1_de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
- link R_pinky_proximal: geometry collision mesh filename=package://dynamic_payload_analysis_core/examples/urdf/h1_de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; visual mesh filename=package://dynamic_payload_analysis_core/examples/urdf/h1_de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
- link R_ring_intermediate: geometry collision mesh filename=package://dynamic_payload_analysis_core/examples/urdf/h1_de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; visual mesh filename=package://dynamic_payload_analysis_core/examples/urdf/h1_de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
- link R_ring_proximal: geometry collision mesh filename=package://dynamic_payload_analysis_core/examples/urdf/h1_de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; visual mesh filename=package://dynamic_payload_analysis_core/examples/urdf/h1_de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
- link R_thumb_distal: geometry collision mesh filename=package://dynamic_payload_analysis_core/examples/urdf/h1_de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; visual mesh filename=package://dynamic_payload_analysis_core/examples/urdf/h1_de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
- link R_thumb_intermediate: geometry collision mesh filename=package://dynamic_payload_analysis_core/examples/urdf/h1_de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; visual mesh filename=package://dynamic_payload_analysis_core/examples/urdf/h1_de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
- link R_thumb_proximal: geometry collision mesh filename=package://dynamic_payload_analysis_core/examples/urdf/h1_de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; visual mesh filename=package://dynamic_payload_analysis_core/examples/urdf/h1_de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
- link R_thumb_proximal_base: geometry collision mesh filename=package://dynamic_payload_analysis_core/examples/urdf/h1_de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; visual mesh filename=package://dynamic_payload_analysis_core/examples/urdf/h1_de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
- link left_ankle_link: geometry collision box size=0.28 0.03 0.024; visual mesh filename=package://dynamic_payload_analysis_core/examples/urdf/h1_de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
- link left_elbow_link: geometry collision cylinder length=0.09 radius=0.03; visual mesh filename=package://dynamic_payload_analysis_core/examples/urdf/h1_de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
- link left_hand_link: geometry collision mesh filename=package://dynamic_payload_analysis_core/examples/urdf/h1_de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; visual mesh filename=package://dynamic_payload_analysis_core/examples/urdf/h1_de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
- link left_hip_pitch_link: geometry collision cylinder length=0.2 radius=0.05; visual mesh filename=package://dynamic_payload_analysis_core/examples/urdf/h1_de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
- link left_hip_roll_link: geometry collision cylinder length=0.01 radius=0.02; visual mesh filename=package://dynamic_payload_analysis_core/examples/urdf/h1_de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
- link left_hip_yaw_link: geometry collision cylinder length=0.02 radius=0.01; visual mesh filename=package://dynamic_payload_analysis_core/examples/urdf/h1_de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
- link left_knee_link: geometry collision cylinder length=0.2 radius=0.05; visual mesh filename=package://dynamic_payload_analysis_core/examples/urdf/h1_de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
- link left_shoulder_pitch_link: geometry collision cylinder length=0.04 radius=0.03; visual mesh filename=package://dynamic_payload_analysis_core/examples/urdf/h1_de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
- link left_shoulder_roll_link: geometry collision cylinder length=0.01 radius=0.04; visual mesh filename=package://dynamic_payload_analysis_core/examples/urdf/h1_de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
- link left_shoulder_yaw_link: geometry collision cylinder length=0.01 radius=0.04; visual mesh filename=package://dynamic_payload_analysis_core/examples/urdf/h1_de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
- link logo_link: geometry visual mesh filename=package://dynamic_payload_analysis_core/examples/urdf/h1_de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
- link pelvis: geometry collision sphere radius=0.05; visual mesh filename=package://dynamic_payload_analysis_core/examples/urdf/h1_de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
- link right_ankle_link: geometry collision box size=0.28 0.03 0.024; visual mesh filename=package://dynamic_payload_analysis_core/examples/urdf/h1_de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
- link right_elbow_link: geometry collision cylinder length=0.09 radius=0.03; visual mesh filename=package://dynamic_payload_analysis_core/examples/urdf/h1_de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
- link right_hand_link: geometry collision mesh filename=package://dynamic_payload_analysis_core/examples/urdf/h1_de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; visual mesh filename=package://dynamic_payload_analysis_core/examples/urdf/h1_de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
- link right_hip_pitch_link: geometry collision cylinder length=0.2 radius=0.05; visual mesh filename=package://dynamic_payload_analysis_core/examples/urdf/h1_de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
- link right_hip_roll_link: geometry collision cylinder length=0.01 radius=0.02; visual mesh filename=package://dynamic_payload_analysis_core/examples/urdf/h1_de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
- link right_hip_yaw_link: geometry collision cylinder length=0.02 radius=0.01; visual mesh filename=package://dynamic_payload_analysis_core/examples/urdf/h1_de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
- link right_knee_link: geometry collision cylinder length=0.2 radius=0.05; visual mesh filename=package://dynamic_payload_analysis_core/examples/urdf/h1_de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
- link right_shoulder_pitch_link: geometry collision cylinder length=0.04 radius=0.03; visual mesh filename=package://dynamic_payload_analysis_core/examples/urdf/h1_de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
- link right_shoulder_roll_link: geometry collision cylinder length=0.01 radius=0.04; visual mesh filename=package://dynamic_payload_analysis_core/examples/urdf/h1_de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
- link right_shoulder_yaw_link: geometry collision cylinder length=0.01 radius=0.04; visual mesh filename=package://dynamic_payload_analysis_core/examples/urdf/h1_de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
- link torso_link: geometry collision box size=0.08 0.16 0.1; visual mesh filename=package://dynamic_payload_analysis_core/examples/urdf/h1_de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
